File: PCB/Tape/V2/Tape_V2.brd (EAGLE design)
At the start: 48.6 x 40.6 mm, 38 parts, among them J1 AUDIO_JACK_3.5MM_PTH, J2 AUDIO_JACK_3.5MM_PTH, T1 2N3904, T10 2N3904, T2 2N3904, T3 2N3904, T4 2N3904, T5 2N3904, T6 2N3904, T7 2N3904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

Commit message: tape board fix
Connections:
- net TAPE_EAR: now also JP1.17; no longer JP1.5
- net TAPE_MIC: now also JP1.19; no longer JP1.7
Routing:
- net TAPE_EAR: track 61.6 -> 75.4 mm
- net TAPE_MIC: track 46.3 -> 56.1 mm
Changed lines of the file:
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@@
 </signal>
 <signal name="TAPE_EAR">
-<contactref element="JP1" pad="5"/>
 <contactref element="R20" pad="2"/>
 <contactref element="T10" pad="1"/>
@@
 <wire x1="32.385" y1="33.655" x2="32.385" y2="39.0525" width="0.2032" layer="16"/>
 <wire x1="46.6725" y1="32.385" x2="46.0375" y2="33.02" width="0.2032" layer="16"/>
-<wire x1="20.6375" y1="8.89" x2="20.6375" y2="13.335" width="0.2032" layer="16"/>
-<wire x1="20.6375" y1="13.335" x2="21.2725" y2="13.97" width="0.2032" layer="16"/>
-<wire x1="21.2725" y1="13.97" x2="21.2725" y2="24.13" width="0.2032" layer="16"/>
-<wire x1="21.2725" y1="24.13" x2="22.225" y2="25.0825" width="0.2032" layer="16"/>
+<wire x1="22.225" y1="25.0825" x2="21.2725" y2="24.13" width="0.2032" layer="16"/>
 <wire x1="22.225" y1="25.0825" x2="26.3525" y2="25.0825" width="0.2032" layer="16"/>
 <via x="26.3525" y="25.0825" extent="1-16" drill="0.35"/>
@@
 <wire x1="32.385" y1="32.7406" x2="32.385" y2="39.0525" width="0.2032" layer="1"/>
 <wire x1="27.7927" y1="32.7406" x2="32.385" y2="32.7406" width="0.2032" layer="1"/>
+<contactref element="JP1" pad="17"/>
+<wire x1="21.2725" y1="10.4775" x2="21.59" y2="10.16" width="0.2032" layer="16"/>
+<wire x1="21.59" y1="10.16" x2="35.2425" y2="10.16" width="0.2032" layer="16"/>
+<wire x1="35.2425" y1="10.16" x2="35.8775" y2="9.525" width="0.2032" layer="16"/>
+<wire x1="35.8775" y1="9.525" x2="35.8775" y2="8.89" width="0.2032" layer="16"/>
+<wire x1="21.2725" y1="24.13" x2="21.2725" y2="10.4775" width="0.2032" layer="16"/>
 </signal>
 <signal name="TAPE_MIC">
-<contactref element="JP1" pad="7"/>
 <contactref element="J2" pad="TIP"/>
 <wire x1="37.2275" y1="35.005" x2="37.2275" y2="33.4175" width="0.2032" layer="1"/>
@@
 <wire x1="21.9075" y1="18.7325" x2="21.2725" y2="18.0975" width="0.2032" layer="1"/>
 <wire x1="21.2725" y1="18.0975" x2="21.2725" y2="13.97" width="0.2032" layer="1"/>
-<wire x1="21.9075" y1="13.335" x2="25.4" y2="13.335" width="0.2032" layer="1"/>
-<wire x1="25.4" y1="13.335" x2="25.7175" y2="13.0175" width="0.2032" layer="1"/>
-<wire x1="25.7175" y1="13.0175" x2="25.7175" y2="10.4775" width="0.2032" layer="1"/>
-<wire x1="25.7175" y1="10.4775" x2="25.4" y2="10.16" width="0.2032" layer="1"/>
-<wire x1="25.4" y1="10.16" x2="23.495" y2="10.16" width="0.2032" layer="1"/>
-<wire x1="23.495" y1="10.16" x2="23.1775" y2="9.8425" width="0.2032" layer="1"/>
-<wire x1="23.1775" y1="9.8425" x2="23.1775" y2="8.89" width="0.2032" layer="1"/>
 <wire x1="37.2275" y1="33.4175" x2="35.8775" y2="32.0675" width="0.2032" layer="1"/>
 <wire x1="28.575" y1="32.0675" x2="27.6225" y2="31.115" width="0.2032" layer="1"/>
-<wire x1="21.2725" y1="13.97" x2="21.9075" y2="13.335" width="0.2032" layer="1"/>
 <via x="35.8775" y="32.0675" extent="1-16" drill="0.35"/>
 <wire x1="35.8775" y1="32.0675" x2="35.56" y2="31.75" width="0.2032" layer="16"/>
@@
 <wire x1="30.6654" y1="31.75" x2="30.3507" y2="32.0647" width="0.2032" layer="1"/>
 <wire x1="30.3507" y1="32.0647" x2="28.5778" y2="32.0647" width="0.2032" layer="1"/>
+<contactref element="JP1" pad="19"/>
+<wire x1="21.2725" y1="13.97" x2="21.59" y2="13.6525" width="0.2032" layer="1"/>
+<wire x1="21.59" y1="13.6525" x2="25.0825" y2="13.6525" width="0.2032" layer="1"/>
+<wire x1="25.0825" y1="13.6525" x2="25.7175" y2="13.0175" width="0.2032" layer="1"/>
+<wire x1="36.0248" y1="10.1219" x2="36.0629" y2="10.16" width="0.2032" layer="1"/>
+<wire x1="36.0629" y1="10.16" x2="37.7825" y2="10.16" width="0.2032" layer="1"/>
+<wire x1="26.3906" y1="10.1219" x2="36.0248" y2="10.1219" width="0.2032" layer="1"/>
+<wire x1="37.7825" y1="10.16" x2="38.4175" y2="9.525" width="0.2032" layer="1"/>
+<wire x1="38.4175" y1="9.525" x2="38.4175" y2="8.89" width="0.2032" layer="1"/>
+<wire x1="25.7175" y1="13.0175" x2="25.7175" y2="10.795" width="0.2032" layer="1"/>
+<wire x1="25.7175" y1="10.795" x2="26.3906" y2="10.1219" width="0.2032" layer="1"/>
 </signal>
 <signal name="N$8">

Commit message: missing resistor
Parts:
- added R22: 3k, adafruit:0204/7
Connections:
- net GND: now also R22.1
- net N$6: now also R22.2
Routing:
- net N$6: track 15.8 -> 33.3 mm
Changed lines of the file:
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@@
 <drawing>
 <settings>
-<setting alwaysvectorfont="no"/>
+<setting alwaysvectorfont="yes"/>
 <setting verticaltext="up"/>
 </settings>
@@
 </element>
 <element name="T6" library="transistor" library_urn="urn:adsk.eagle:library:402" package="TO92" package3d_urn="urn:adsk.eagle:package:28523/2" value="2N3904" x="13.6525" y="30.1625" smashed="yes" rot="R180">
-<attribute name="NAME" x="10.4775" y="29.845" size="1.27" layer="25" ratio="10" rot="R180"/>
+<attribute name="NAME" x="16.1925" y="27.94" size="1.27" layer="25" ratio="10" rot="R180"/>
 <attribute name="POPULARITY" value="27" x="13.6525" y="30.1625" size="1.778" layer="27" rot="R180" display="off"/>
 <attribute name="VALUE" x="10.4775" y="31.4325" size="1.27" layer="27" ratio="10" rot="R180"/>
@@
 <attribute name="NAME" x="45.6946" y="26.3525" size="0.9906" layer="25" ratio="12" rot="R90"/>
 <attribute name="VALUE" x="47.1551" y="25.6794" size="0.9906" layer="27" ratio="12" rot="R90"/>
+</element>
+<element name="R22" library="adafruit" library_urn="urn:adsk.eagle:library:420" package="0204/7" package3d_urn="urn:adsk.eagle:package:6240596/1" value="3k" x="8.255" y="26.9875" smashed="yes" rot="R270">
+<attribute name="NAME" x="10.4521" y="26.035" size="0.9906" layer="25" ratio="12" rot="R90"/>
+<attribute name="VALUE" x="7.7724" y="28.6131" size="0.9906" layer="27" ratio="12" rot="R270"/>
 </element>
 </elements>
@@
 <contactref element="T10" pad="3"/>
 <contactref element="T9" pad="3"/>
+<contactref element="R22" pad="1"/>
 </signal>
 <signal name="N$1">
@@
 <contactref element="R2" pad="2"/>
 <wire x1="5.3975" y1="26.67" x2="5.3975" y2="24.4475" width="0.2032" layer="1"/>
-<wire x1="5.3975" y1="24.4475" x2="7.9375" y2="24.4475" width="0.2032" layer="1"/>
-<wire x1="7.9375" y1="24.4475" x2="8.89" y2="23.495" width="0.2032" layer="1"/>
-<wire x1="8.89" y1="23.495" x2="8.89" y2="18.7325" width="0.2032" layer="1"/>
+<wire x1="6.6675" y1="18.7325" x2="5.3975" y2="20.0025" width="0.2032" layer="1"/>
+<wire x1="5.3975" y1="24.4475" x2="5.3975" y2="20.0025" width="0.2032" layer="1"/>
+<wire x1="8.89" y1="18.7325" x2="6.6675" y2="18.7325" width="0.2032" layer="1"/>
 </signal>
 <signal name="N$4">
@@
 <wire x1="13.6525" y1="10.795" x2="10.4775" y2="7.62" width="0.2032" layer="1"/>
 <wire x1="23.1775" y1="10.795" x2="13.6525" y2="10.795" width="0.2032" layer="1"/>
+<contactref element="R22" pad="2"/>
+<wire x1="10.4775" y1="7.62" x2="10.16" y2="7.9375" width="0.2032" layer="16"/>
+<wire x1="10.16" y1="7.9375" x2="10.16" y2="11.43" width="0.2032" layer="16"/>
+<wire x1="7.3025" y1="14.2875" x2="7.3025" y2="22.5425" width="0.2032" layer="16"/>
+<wire x1="7.3025" y1="22.5425" x2="7.9375" y2="23.1775" width="0.2032" layer="16"/>
+<wire x1="7.9375" y1="23.1775" x2="8.255" y2="23.1775" width="0.2032" layer="16"/>
+<wire x1="10.16" y1="11.43" x2="7.3025" y2="14.2875" width="0.2032" layer="16"/>
 </signal>
 <signal name="N$5">
