File: PCB/Tape/V2/Tape_V2.sch (EAGLE design)
At the start: 38 parts, among them J1 AUDIO_JACK_3.5MM_PTH, J2 AUDIO_JACK_3.5MM_PTH, T1 2N3904, T10 2N3904, T2 2N3904, T3 2N3904, T4 2N3904, T5 2N3904, T6 2N3904, T7 2N3904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

Commit message: tape board fix
Connections:
- net TAPE_EAR: now also JP1.17; no longer JP1.5
- net TAPE_MIC: now also JP1.19; no longer JP1.7
Changed lines of the file:
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@@
 <net name="TAPE_EAR" class="0">
-<segment>
-<pinref part="JP1" gate="A" pin="5"/>
-<wire x1="27.94" y1="33.02" x2="12.7" y2="33.02" width="0.1524" layer="91"/>
-<label x="10.16" y="33.02" size="1.778" layer="95"/>
-</segment>
 <segment>
 <pinref part="R20" gate="G$1" pin="2"/>
@@
 <label x="236.22" y="101.6" size="1.778" layer="95"/>
 </segment>
+<segment>
+<pinref part="JP1" gate="A" pin="17"/>
+<wire x1="27.94" y1="17.78" x2="10.16" y2="17.78" width="0.1524" layer="91"/>
+<label x="10.16" y="17.78" size="1.778" layer="95"/>
+</segment>
 </net>
 <net name="TAPE_MIC" class="0">
-<segment>
-<pinref part="JP1" gate="A" pin="7"/>
-<wire x1="27.94" y1="30.48" x2="12.7" y2="30.48" width="0.1524" layer="91"/>
-<label x="10.16" y="30.48" size="1.778" layer="95"/>
-</segment>
 <segment>
 <pinref part="J2" gate="G$1" pin="TIP"/>
@@
 <label x="45.72" y="109.22" size="1.778" layer="95"/>
 </segment>
+<segment>
+<pinref part="JP1" gate="A" pin="19"/>
+<wire x1="27.94" y1="15.24" x2="10.16" y2="15.24" width="0.1524" layer="91"/>
+<label x="10.16" y="15.24" size="1.778" layer="95"/>
+</segment>
 </net>

Commit message: missing resistor
Parts:
- added R22: 3k, adafruit:R-US_0204/7
Connections:
- net GND: now also R22.1
- net N$6: now also R22.2
Changed lines of the file:
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@@
 <part name="R20" library="adafruit" library_urn="urn:adsk.eagle:library:420" deviceset="R-US_" device="0204/7" package3d_urn="urn:adsk.eagle:package:6240596/1" value="1k"/>
 <part name="GND15" library="SparkFun-PowerSymbols" library_urn="urn:adsk.eagle:library:530" deviceset="GND" device=""/>
+<part name="R22" library="adafruit" library_urn="urn:adsk.eagle:library:420" deviceset="R-US_" device="0204/7" package3d_urn="urn:adsk.eagle:package:6240596/1" value="3k"/>
 </parts>
 <sheets>
@@
 <attribute name="VALUE" x="111.76" y="65.786" size="1.778" layer="96" align="top-center"/>
 </instance>
-<instance part="GND9" gate="1" x="53.34" y="53.34" smashed="yes">
-<attribute name="VALUE" x="53.34" y="53.086" size="1.778" layer="96" align="top-center"/>
+<instance part="GND9" gate="1" x="81.28" y="50.8" smashed="yes">
+<attribute name="VALUE" x="81.28" y="50.546" size="1.778" layer="96" align="top-center"/>
 </instance>
 <instance part="T4" gate="G1" x="121.92" y="86.36" smashed="yes">
@@
 <instance part="GND15" gate="1" x="180.34" y="81.28" smashed="yes">
 <attribute name="VALUE" x="180.34" y="81.026" size="1.778" layer="96" align="top-center"/>
+</instance>
+<instance part="R22" gate="G$1" x="81.28" y="58.42" smashed="yes" rot="R90">
+<attribute name="NAME" x="79.7814" y="54.61" size="1.778" layer="95" rot="R90"/>
+<attribute name="VALUE" x="84.582" y="54.61" size="1.778" layer="96" rot="R90"/>
 </instance>
 </instances>
@@
 <pinref part="GND15" gate="1" pin="GND"/>
 </segment>
+<segment>
+<pinref part="R22" gate="G$1" pin="1"/>
+<pinref part="GND9" gate="1" pin="GND"/>
+</segment>
 </net>
 <net name="N$1" class="0">
@@
 <pinref part="T2" gate="G1" pin="B"/>
 <wire x1="76.2" y1="66.04" x2="81.28" y2="66.04" width="0.1524" layer="91"/>
-</segment>
-</net>
+<pinref part="R22" gate="G$1" pin="2"/>
+<wire x1="81.28" y1="63.5" x2="81.28" y2="66.04" width="0.1524" layer="91"/>
+<junction x="81.28" y="66.04"/>
+</segment>
+</net>
