File: PCB/TMS Card/XPL-32 - Copy - Copy.brd (EAGLE design)
At the start: 101.3 x 80 mm, 23 parts, among them IC1 74HC138N, IC2 74HCT04N, IC4 74LS00N, T2 2N2222

Commit message: Time to make z cir cut bord!!!!
Routing:
- net RAS: track 0.00 -> 30.3 mm, vias 0 -> 2
Changed lines of the file:
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@@
 <contactref element="VDP" pad="1"/>
 <contactref element="IC2" pad="5"/>
-<wire x1="13.97" y1="20.32" x2="6.35" y2="43.18" width="0" layer="19" extent="1-1"/>
+<wire x1="13.97" y1="20.32" x2="12.065" y2="20.32" width="0.1524" layer="16"/>
+<wire x1="12.065" y1="20.32" x2="11.43" y2="20.955" width="0.1524" layer="16"/>
+<wire x1="11.43" y1="20.955" x2="11.43" y2="26.67" width="0.1524" layer="16"/>
+<wire x1="11.43" y1="26.67" x2="12.065" y2="27.305" width="0.1524" layer="16"/>
+<via x="12.065" y="27.305" extent="1-16" drill="0.35"/>
+<wire x1="12.065" y1="27.305" x2="12.065" y2="35.56" width="0.1524" layer="1"/>
+<via x="12.065" y="35.56" extent="1-16" drill="0.35"/>
+<wire x1="12.065" y1="35.56" x2="7.62" y2="35.56" width="0.1524" layer="16"/>
+<wire x1="7.62" y1="35.56" x2="6.35" y2="36.83" width="0.1524" layer="16"/>
+<wire x1="6.35" y1="36.83" x2="6.35" y2="43.18" width="0.1524" layer="16"/>
 </signal>
 <signal name="CAS">
