File: PCB/XPL-32/XPL-32.sch (EAGLE design)
At the start: 81 parts, among them IC10 MCP120-450DI_TO, IC4 74HC00N, IC7 74HC138N, IC8 328P, IC9 74HCT166N, J3 973, J4 AUDIO_JACK_3.5MM_PTH, K1 APF30205C, U1 W65C02SP, U3 328P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

Commit message: fix
Other:
- note added: "By Waverider"
- note removed: "By Liam Oppenheimer"
Changed lines of the file:
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@@
 <?xml version="1.0" encoding="utf-8"?>
 <!DOCTYPE eagle SYSTEM "eagle.dtd">
-<eagle version="9.6.0">
+<eagle version="9.6.2">
 <drawing>
 <settings>
@@
 <plain>
 <text x="154.94" y="-53.34" size="5.08" layer="94">XPL-32</text>
-<text x="180.34" y="-53.34" size="5.08" layer="94">By Liam Oppenheimer</text>
+<text x="180.34" y="-53.34" size="5.08" layer="94">By Waverider</text>
 <text x="241.3" y="-66.04" size="3.81" layer="94">A</text>
 <text x="-111.76" y="165.1" size="1.778" layer="97">VIDEO/EXTVID Relay</text>
