File: PCB/kicad/sd/v2/memory card/memory card.kicad_pcb (KiCad board)
At the start: 2 copper layers, 48.5 x 33 mm, 11 parts, among them IC2 74LVC125APW,112, J2 DM3AT-SF-PEJM5_40_, J3 PINHD_1x6_Male, U1 AMS1117

Commit message: me and xat - WE DID IT.
sd saving fixed

i think.
Routing:
- net SCK: track 54.9 -> 53.5 mm
